Commit message: Added LiDAR sensor

File: quadruped/quadruped.urdf (robot description, URDF)
Before this commit: robot quadruped, 13 links, 12 joints
Links:
- added link lidar1, mass 0.01926679869584365; collision mesh filename=meshes/lidar1.stl scale=0.001 0.001 0.001; visual mesh filename=meshes/lidar1.stl scale=0.001 0.001 0.001
- link base_link: mass 44.76275372212462 -> 10.0
- link calfBL1: mass 0.45030095449806384 -> 2.0
- link calfBR1: mass 0.45030095449806384 -> 2.0
- link calfFL1: mass 0.45030095449806384 -> 2.0
- link calfFR1: mass 0.45030095449806384 -> 2.0
- link hipBL1: mass 1.459703797805085 -> 0.5
- link hipBR1: mass 1.459703797805085 -> 0.5
- link hipFL1: mass 1.459703797805085 -> 0.5
- link hipFR1: mass 1.459703797805085 -> 0.5
- link legBR1: mass 0.5177742031085164 -> 1.0
- link legBl1: mass 0.5177742031085164 -> 1.0
- link legFL1: mass 0.5177742031085164 -> 1.0
- link legFR1: mass 0.5177742031085164 -> 1.0
Joints:
- added joint Rigid_14: type fixed, parent base_link, child lidar1, origin xyz=0.0 -0.425898 0.569105 rpy=0 0 -1.57079632679

Commit message: Add Some DRL Loop Logic

File: quadruped/quadruped.urdf (robot description, URDF)
Before this commit: robot quadruped, 14 links, 13 joints
Links:
- link base_link: mass 10.0 -> 7.5
- link calfBL1: mass 2.0 -> 2.5
- link calfBR1: mass 2.0 -> 2.5
- link calfFL1: mass 2.0 -> 2.5
- link calfFR1: mass 2.0 -> 2.5
- link legBR1: mass 1.0 -> 2.5
- link legBl1: mass 1.0 -> 2.5
- link legFL1: mass 1.0 -> 2.5
- link legFR1: mass 1.0 -> 2.5
- link lidar1: mass 0.01926679869584365 -> 0.02
Joints:
- joint Revolute_11: axis 1.0 -0.0 0.0 -> 1.0 -0.0 -0.0
- joint Rigid_14: origin xyz=0.0 -0.425898 0.569105 rpy=0 0 -1.57079632679 -> xyz=0.0 -0.575898 -0.380895 rpy=0 0 0
- joint hipjointBL: origin xyz=0.095003 0.374102 0.474105 rpy=0 0 0 -> xyz=0.095003 0.299102 -0.000895 rpy=0 0 0
- joint hipjointBR: origin xyz=-0.094997 0.374102 0.474105 rpy=0 0 0 -> xyz=-0.094997 0.299102 -0.000895 rpy=0 0 0
- joint hipjointFL: origin xyz=0.095003 -0.225898 0.474105 rpy=0 0 0 -> xyz=0.095003 -0.300898 -0.000895 rpy=0 0 0
- joint hipjointFR: origin xyz=-0.094997 -0.225898 0.474105 rpy=0 0 0 -> xyz=-0.094997 -0.300898 -0.000895 rpy=0 0 0

Commit message: Add reward/done function

File: quadruped/quadruped.urdf (robot description, URDF)
Before this commit: robot quadruped, 14 links, 13 joints
Links:
- link base_link: mass 7.5 -> 5.0
